File: cansat.kicad_pcb (KiCad board)
At the start: 2 copper layers, 50 x 50 mm, 4 parts

Commit message: draft 3 pcb chn
Parts:
- moved U2 9.91 mm to (112.0, 71.4)
Routing:
- net Net-(A1-SDA/A4): track 39.0 -> 50.9 mm, vias 0 -> 1
- net Net-(A1-SCL/A5): track 42.6 -> 54.4 mm, vias 0 -> 1
- net +5V: track 56.6 -> 59.7 mm
Changed lines of the file:
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@@
 	(footprint "GovindLibrary:BMP280"
 		(layer "F.Cu")
-		(at 111.633 81.28 -90)
+		(at 112.014 71.374 -90)
 		(property "Reference" "U2"
 			(at 0 -0.254 270)
@@
 			(unlocked yes)
 			(layer "F.Fab")
+			(hide yes)
 			(effects
 				(font
@@
 			(stroke
 				(width 0.1)
-				(type default)
+				(type solid)
 			)
 			(fill no)
-			(layer "F.SilkS")
+			(layer "F.CrtYd")
 		)
 		(fp_text user "Gnd"
@@
 			(unlocked yes)
 			(layer "F.Fab")
+			(hide yes)
 			(effects
 				(font
@@
 			(stroke
 				(width 0.1)
-				(type default)
+				(type solid)
 			)
 			(fill no)
-			(layer "F.SilkS")
+			(layer "F.CrtYd")
 		)
 		(fp_text user "XCL"
@@
 			(unlocked yes)
 			(layer "F.Fab")
+			(hide yes)
 			(effects
 				(font
@@
 			(stroke
 				(width 0.1)
-				(type default)
+				(type solid)
 			)
 			(fill no)
-			(layer "F.SilkS")
+			(layer "F.CrtYd")
 		)
 		(fp_text user "PPS"
@@
 		)
 		(property "Value" "Arduino_Nano_Every"
-			(at 8.89 19.05 90)
-			(layer "F.Fab")
-			(effects
-				(font
-					(size 1 1)
-					(thickness 0.15)
+			(at 7.62 -2.4096 180)
+			(layer "F.SilkS")
+			(effects
+				(font
+					(size 1 1)
+					(thickness 0.2)
+					(bold yes)
 				)
 			)
@@
 	)
 	(gr_rect
+		(start 108.712 64.8208)
+		(end 120.904 80.2132)
+		(stroke
+			(width 0.1)
+			(type default)
+		)
+		(fill no)
+		(layer "F.SilkS")
+	)
+	(gr_rect
+		(start 92.1004 92.4052)
+		(end 122.2756 113.1316)
+		(stroke
+			(width 0.1)
+			(type default)
+		)
+		(fill no)
+		(layer "F.SilkS")
+	)
+	(gr_rect
+		(start 92.3544 64.6684)
+		(end 106.7816 80.2132)
+		(stroke
+			(width 0.1)
+			(type solid)
+		)
+		(fill no)
+		(layer "F.SilkS")
+	)
+	(gr_rect
 		(start 91.44 64.008)
-		(end 141.478 114.046)
+		(end 141.44 114.008)
 		(stroke
 			(width 0.2)
@@
 	)
 	(segment
-		(start 121.666 83.439)
-		(end 121.793 83.439)
+		(start 109.474 91.186)
+		(end 120.65 91.186)
+		(width 0.2)
+		(layer "F.Cu")
+		(net 1)
+	)
+	(segment
+		(start 121.666 90.17)
+		(end 121.666 83.08)
+		(width 0.2)
+		(layer "F.Cu")
+		(net 1)
+	)
+	(segment
+		(start 109.474 91.186)
+		(end 96.901 78.613)
+		(width 0.2)
+		(layer "F.Cu")
+		(net 1)
+	)
+	(segment
+		(start 121.666 83.08)
+		(end 124.085 83.08)
 		(width 0.2)
 		(layer "F.Cu")
@@
 	)
 	(segment
-		(start 109.474 91.186)
-		(end 120.65 91.186)
-		(width 0.2)
-		(layer "F.Cu")
-		(net 1)
-	)
-	(segment
-		(start 121.793 83.439)
-		(end 122.152 83.08)
-		(width 0.2)
-		(layer "F.Cu")
-		(net 1)
-	)
-	(segment
-		(start 121.666 90.17)
-		(end 121.666 83.439)
-		(width 0.2)
-		(layer "F.Cu")
-		(net 1)
-	)
-	(segment
-		(start 122.152 83.08)
-		(end 124.085 83.08)
-		(width 0.2)
-		(layer "F.Cu")
-		(net 1)
-	)
-	(segment
-		(start 96.901 78.613)
-		(end 109.474 91.186)
-		(width 0.2)
-		(layer "F.Cu")
-		(net 1)
+		(start 121.066 85.979)
+		(end 121.066 89.5)
+		(width 0.2)
+		(layer "F.Cu")
+		(net 5)
+	)
+	(segment
+		(start 121.066 89.5)
+		(end 120.365 90.201)
+		(width 0.2)
+		(layer "F.Cu")
+		(net 5)
 	)
 	(segment
 		(start 120.365 90.201)
-		(end 121.066 89.5)
+		(end 111.029 90.201)
 		(width 0.2)
 		(layer "F.Cu")
@@
 	)
 	(segment
-		(start 99.441 78.613)
-		(end 99.949 78.613)
-		(width 0.2)
-		(layer "F.Cu")
-		(net 5)
-	)
-	(segment
-		(start 111.537 90.201)
-		(end 120.365 90.201)
-		(width 0.2)
-		(layer "F.Cu")
-		(net 5)
-	)
-	(segment
-		(start 100.076 78.74)
-		(end 111.537 90.201)
-		(width 0.2)
-		(layer "F.Cu")
-		(net 5)
-	)
-	(segment
-		(start 121.066 89.5)
-		(end 121.066 85.979)
-		(width 0.2)
-		(layer "F.Cu")
-		(net 5)
-	)
-	(segment
-		(start 99.949 78.613)
-		(end 100.076 78.74)
+		(start 111.029 90.201)
+		(end 99.441 78.613)
 		(width 0.2)
 		(layer "F.Cu")
@@
 	)
 	(segment
-		(start 119.253 81.28)
-		(end 119.614 81.641)
+		(start 139.325 85.62)
+		(end 128.064 74.359)
 		(width 0.2)
 		(layer "F.Cu")
@@
 	)
 	(segment
-		(start 119.614 81.641)
-		(end 135.346 81.641)
+		(start 119.634 71.374)
+		(end 122.619 74.359)
 		(width 0.2)
 		(layer "F.Cu")
@@
 	)
 	(segment
-		(start 135.346 81.641)
-		(end 139.325 85.62)
+		(start 103.632 93.599)
+		(end 107.335235 89.895765)
 		(width 0.2)
 		(layer "F.Cu")
@@
 	)
 	(segment
-		(start 119.253 81.28)
-		(end 115.951 81.28)
-		(width 0.2)
-		(layer "B.Cu")
+		(start 122.619 74.359)
+		(end 128.064 74.359)
+		(width 0.2)
+		(layer "F.Cu")
 		(net 8)
 	)
-	(segment
-		(start 115.951 81.28)
-		(end 103.632 93.599)
-		(width 0.2)
-		(layer "B.Cu")
+	(via
+		(at 107.335235 89.895765)
+		(size 0.6)
+		(drill 0.3)
+		(layers "F.Cu" "B.Cu")
 		(net 8)
 	)
 	(segment
-		(start 119.253 76.2)
-		(end 119.888 76.835)
+		(start 107.335235 83.672765)
+		(end 119.634 71.374)
+		(width 0.2)
+		(layer "B.Cu")
+		(net 8)
+	)
+	(segment
+		(start 107.335235 89.895765)
+		(end 107.335235 83.672765)
+		(width 0.2)
+		(layer "B.Cu")
+		(net 8)
+	)
+	(segment
+		(start 124.968 65.532)
+		(end 120.396 65.532)
+		(width 0.4)
+		(layer "B.Cu")
+		(net 15)
+	)
+	(segment
+		(start 129.816 70.38)
+		(end 124.968 65.532)
+		(width 0.4)
+		(layer "B.Cu")
+		(net 15)
+	)
+	(segment
+		(start 120.396 65.532)
+		(end 119.634 66.294)
 		(width 0.2)
 		(layer "B.Cu")
@@
 		(start 104.521 78.613)
 		(end 104.521 87.63)
-		(width 0.2)
+		(width 0.4)
 		(layer "B.Cu")
 		(net 15)
 	)
 	(segment
+		(start 119.634 66.294)
+		(end 107.315 78.613)
+		(width 0.4)
+		(layer "B.Cu")
+		(net 15)
+	)
+	(segment
 		(start 139.325 70.38)
-		(end 135.664 74.041)
-		(width 0.2)
+		(end 129.816 70.38)
+		(width 0.4)
 		(layer "B.Cu")
 		(net 15)
 	)
 	(segment
-		(start 104.521 78.613)
-		(end 116.84 78.613)
-		(width 0.2)
-		(layer "B.Cu")
-		(net 15)
-	)
-	(segment
-		(start 121.412 74.041)
-		(end 119.253 76.2)
-		(width 0.2)
+		(start 107.315 78.613)
+		(end 104.521 78.613)
+		(width 0.4)
 		(layer "B.Cu")
 		(net 15)
@@
 		(start 104.521 87.63)
 		(end 98.552 93.599)
-		(width 0.2)
+		(width 0.4)
 		(layer "B.Cu")
 		(net 15)
 	)
 	(segment
-		(start 116.84 78.613)
-		(end 119.253 76.2)
-		(width 0.2)
-		(layer "B.Cu")
-		(net 15)
-	)
-	(segment
-		(start 135.664 74.041)
-		(end 121.412 74.041)
-		(width 0.2)
-		(layer "B.Cu")
-		(net 15)
+		(start 127.403 88.16)
+		(end 125.984 86.741)
+		(width 0.2)
+		(layer "F.Cu")
+		(net 16)
+	)
+	(segment
+		(start 139.325 88.16)
+		(end 127.403 88.16)
+		(width 0.2)
+		(layer "F.Cu")
+		(net 16)
+	)
+	(via
+		(at 125.984 86.741)
+		(size 0.6)
+		(drill 0.3)
+		(layers "F.Cu" "B.Cu")
+		(net 16)
+	)
+	(segment
+		(start 118.333 75.215)
+		(end 119.634 73.914)
+		(width 0.2)
+		(layer "B.Cu")
+		(net 16)
 	)
 	(segment
@@
 	)
 	(segment
-		(start 135.346 84.181)
-		(end 139.325 88.16)
+		(start 115.951 83.82)
+		(end 118.333 81.438)
 		(width 0.2)
 		(layer "B.Cu")
@@
 	)
 	(segment
-		(start 119.253 83.82)
+		(start 118.333 81.438)
+		(end 118.333 75.215)
+		(width 0.2)
+		(layer "B.Cu")
+		(net 16)
+	)
+	(segment
+		(start 125.984 86.741)
+		(end 118.872 86.741)
+		(width 0.2)
+		(layer "B.Cu")
+		(net 16)
+	)
+	(segment
+		(start 119.634 73.914)
+		(end 119.995 74.275)
+		(width 0.2)
+		(layer "B.Cu")
+		(net 16)
+	)
+	(segment
+		(start 118.872 86.741)
 		(end 115.951 83.82)
-		(width 0.2)
-		(layer "B.Cu")
-		(net 16)
-	)
-	(segment
-		(start 119.253 83.82)
-		(end 119.614 84.181)
-		(width 0.2)
-		(layer "B.Cu")
-		(net 16)
-	)
-	(segment
-		(start 119.614 84.181)
-		(end 135.346 84.181)
 		(width 0.2)
 		(layer "B.Cu")
@@
 		(polygon
 			(pts
-				(xy 87.503 61.849) (xy 88.519 117.094) (xy 147.447 117.221) (xy 144.399 60.96)
-			)
-		)
+				(xy 87.503 61.849) (xy 88.519 117.094) (xy 144.907 116.713) (xy 144.399 60.96)
+			)
+		)
