File: cansat.kicad_sch (KiCad schematic)
At the start: 1 part

Commit message: draft 1
Parts:
- added U1: ~, symbol New_Library:MPU-6050
- added U2: ~, GovindLibrary:BMP280, symbol New_Library:Bmp-280
- added U3: ~, GovindLibrary:NEO-6m, symbol New_Library:Neo_6-m
Connections:
- net at A1.23 (SDA/A4): now also U1.4 (sda), U2.4 (SDA)
- net at A1.24 (SCL/A5): now also U1.3 (SCL), U2.3 (SCL)
- net GND: now reaches A1.29 (GND), A1.4 (GND)
- net GND: now also U2.2 (Gnd), U3.2 (Gnd)
- net +5V: now reaches A1.30 (VIN)
- net +5V: now also U1. (Vcc), U1.2 (Gnd), U2.1 (Vcc), U3.1 (Vcc)
- net at A1.6 (D3): now also U3.4 (RX)
- net at A1.7 (D4): now also U3.3 (TX)
- no-connect marks 0 -> 29

Commit message: draft 2 sch chn
Parts:
- removed U1: ~, symbol New_Library:MPU-6050
- removed U3: ~, GovindLibrary:NEO-6m, symbol New_Library:Neo_6-m
- added U1: ~, symbol New_Library:Neo_6-m
- added U3: ~, symbol New_Library:MPU-6050
- U2: footprint GovindLibrary:BMP280 -> (none)
Connections:
- net +5V: now also U1.1 (Vcc), U3. (Vcc)
- net GND: now also U1.2 (Gnd), U3.2 (Gnd)
- net SDA: now reaches A1.23 (SDA/A4), U2.4 (SDA)
- net SDA: now also U3.4 (SDA)
- net SCL: now reaches A1.24 (SCL/A5), U2.3 (SCL)
- net SCL: now also U3.3 (SCL)
- net RX: now reaches A1.6 (D3)
- net RX: now also U1.4 (RX)
- net TX: now reaches A1.7 (D4)
- net TX: now also U1.3 (TX)
Other:
- note added: "Arduino nano"
- note added: "BMP-280"
- note added: "MPU-6050"
- note added: "NEO-6M"

Commit message: draft 4 sch chn
Parts:
- added U4: ~, GovindLibrary:Lora module, symbol New_Library:lora_module
- U1: footprint (none) -> GovindLibrary:NEO-6m
- U2: footprint (none) -> GovindLibrary:BMP280
- U3: footprint (none) -> GovindLibrary:MPU-6050
Connections:
- net +5V: now also U4.7 (VCC)
- net GND: now also U4.6 (GND)
- no-connect marks 29 -> 35
Other:
- note added: "LORA Module"
